Commit message: fix: properly handle fastdds version based on rosdistro

File: launch_ext/config/fastdds_profile.xml.xacro (robot description, xacro)
@@ -5,5 +5,7 @@
     <xacro:arg name="own_ip" default="" />
     <xacro:arg name="discovery_protocol" default="CLIENT" />
+    <xacro:arg name="ros_distro" default="jazzy" />
     <xacro:property name="discovery_protocol" value="$(arg discovery_protocol)" />
+    <xacro:property name="ros_distro" value="$(arg ros_distro)" />
     <profiles>
         <transport_descriptors>
@@ -39,14 +41,26 @@
                             <discoveryProtocol>$(arg discovery_protocol)</discoveryProtocol>
                             <discoveryServersList>
-                                <RemoteServer prefix="44.53.00.5f.45.50.52.4f.53.49.4d.41">
-                                    <metatrafficUnicastLocatorList>
-                                        <locator>
-                                            <udpv4>
-                                                <address>$(arg discovery_server_ip)</address>
-                                                <port>11811</port>
-                                            </udpv4>
-                                        </locator>
-                                    </metatrafficUnicastLocatorList>
-                                </RemoteServer>
+                                <!-- FastDDS 3.x (kilted) uses direct locator format -->
+                                <xacro:if value="${ros_distro == 'kilted'}">
+                                    <locator>
+                                        <udpv4>
+                                            <address>$(arg discovery_server_ip)</address>
+                                            <port>11811</port>
+                                        </udpv4>
+                                    </locator>
+                                </xacro:if>
+                                <!-- FastDDS 2.x (jazzy and older) uses RemoteServer wrapper format -->
+                                <xacro:unless value="${ros_distro == 'kilted'}">
+                                    <RemoteServer prefix="44.53.00.5f.45.50.52.4f.53.49.4d.41">
+                                        <metatrafficUnicastLocatorList>
+                                            <locator>
+                                                <udpv4>
+                                                    <address>$(arg discovery_server_ip)</address>
+                                                    <port>11811</port>
+                                                </udpv4>
+                                            </locator>
+                                        </metatrafficUnicastLocatorList>
+                                    </RemoteServer>
+                                </xacro:unless>
                             </discoveryServersList>
                         </discovery_config>

Commit message: add server config to profile

File: launch_ext/config/fastdds_profile.xml.xacro (robot description, xacro)
@@ -9,4 +9,5 @@
     <xacro:property name="discovery_protocol" value="$(arg discovery_protocol)" />
     <xacro:property name="ros_distro" value="$(arg ros_distro)" />
+    <xacro:property name="own_ip" value="$(arg own_ip)" />
     <profiles>
         <transport_descriptors>
@@ -21,9 +22,11 @@
                 <transport_id>udp_transport</transport_id>
                 <type>UDPv4</type>
-                <interfaces>
-                    <allowlist>
-                        <interface name="$(arg own_ip)" netmask_filter="OFF" />
-                    </allowlist>
-                </interfaces>
+                <xacro:if value="${own_ip != '0.0.0.0'}">
+                    <interfaces>
+                        <allowlist>
+                            <interface name="$(arg own_ip)" netmask_filter="OFF" />
+                        </allowlist>
+                    </interfaces>
+                </xacro:if>
             </transport_descriptor>
         </transport_descriptors>
@@ -42,5 +45,20 @@
                 </defaultUnicastLocatorList>
                 <useBuiltinTransports>false</useBuiltinTransports>
-                <xacro:if value="${discovery_protocol != 'SIMPLE'}">
+                <xacro:if value="${discovery_protocol == 'SERVER'}">
+                    <builtin>
+                        <discovery_config>
+                            <discoveryProtocol>SERVER</discoveryProtocol>
+                        </discovery_config>
+                        <metatrafficUnicastLocatorList>
+                            <locator>
+                                <udpv4>
+                                    <address>$(arg own_ip)</address>
+                                    <port>11811</port>
+                                </udpv4>
+                            </locator>
+                        </metatrafficUnicastLocatorList>
+                    </builtin>
+                </xacro:if>
+                <xacro:if value="${discovery_protocol != 'SIMPLE' and discovery_protocol != 'SERVER'}">
                     <builtin>
                         <discovery_config>

Commit message: add allowed_interfaces list

File: launch_ext/config/fastdds_profile.xml.xacro (robot description, xacro)
@@ -4,10 +4,33 @@
     <xacro:arg name="discovery_server_ip" default="" />
     <xacro:arg name="launch_log_dir" default="" />
-    <xacro:arg name="own_ip" default="" />
+    <xacro:arg name="allowed_interfaces" default="" />
     <xacro:arg name="discovery_protocol" default="CLIENT" />
     <xacro:arg name="ros_distro" default="jazzy" />
     <xacro:property name="discovery_protocol" value="$(arg discovery_protocol)" />
     <xacro:property name="ros_distro" value="$(arg ros_distro)" />
-    <xacro:property name="own_ip" value="$(arg own_ip)" />
+    <xacro:property name="iface_list" value="${'$(arg allowed_interfaces)'.split()}" />
+    <!-- Recursive macro to emit allowlist interface entries -->
+    <xacro:macro name="allowlist_loop" params="ifaces:=^">
+        <xacro:if value="${ifaces}">
+            <xacro:property name="iface" value="${ifaces.pop(0)}"/>
+            <interface name="${iface}" netmask_filter="OFF" />
+            <xacro:allowlist_loop/>
+        </xacro:if>
+    </xacro:macro>
+    <!-- Recursive macro to emit locator entries -->
+    <xacro:macro name="locator_loop" params="addrs:=^ port:=0">
+        <xacro:if value="${addrs}">
+            <xacro:property name="addr" value="${addrs.pop(0)}"/>
+            <locator>
+                <udpv4>
+                    <address>${addr}</address>
+                    <xacro:if value="${port != 0}">
+                        <port>${port}</port>
+                    </xacro:if>
+                </udpv4>
+            </locator>
+            <xacro:locator_loop/>
+        </xacro:if>
+    </xacro:macro>
     <profiles>
         <transport_descriptors>
@@ -22,10 +45,8 @@
                 <transport_id>udp_transport</transport_id>
                 <type>UDPv4</type>
-                <xacro:if value="${own_ip != '0.0.0.0'}">
+                <xacro:if value="${iface_list}">
                     <interfaces>
                         <allowlist>
-                            <interface name="$(arg own_ip)" netmask_filter="OFF" />
-                            <!-- TODO: remove hardcoded tailscale interface after testing -->
-                            <interface name="100.64.0.170" netmask_filter="OFF" />
+                            <xacro:allowlist_loop ifaces="${list(iface_list)}"/>
                         </allowlist>
                     </interfaces>
@@ -39,11 +60,9 @@
                     <transport_id>udp_transport</transport_id>
                 </userTransports>
-                <defaultUnicastLocatorList>
-                    <locator>
-                        <udpv4>
-                            <address>$(arg own_ip)</address>
-                        </udpv4>
-                    </locator>
-                </defaultUnicastLocatorList>
+                <xacro:if value="${iface_list}">
+                    <defaultUnicastLocatorList>
+                        <xacro:locator_loop addrs="${list(iface_list)}"/>
+                    </defaultUnicastLocatorList>
+                </xacro:if>
                 <useBuiltinTransports>false</useBuiltinTransports>
                 <xacro:if value="${discovery_protocol == 'SERVER'}">
@@ -53,17 +72,15 @@
                         </discovery_config>
                         <metatrafficUnicastLocatorList>
-                            <locator>
-                                <udpv4>
-                                    <address>$(arg own_ip)</address>
-                                    <port>11811</port>
-                                </udpv4>
-                            </locator>
-                            <!-- TODO: remove hardcoded tailscale locator after testing -->
-                            <locator>
-                                <udpv4>
-                                    <address>100.64.0.170</address>
-                                    <port>11811</port>
-                                </udpv4>
-                            </locator>
+                            <xacro:if value="${iface_list}">
+                                <xacro:locator_loop addrs="${list(iface_list)}" port="11811"/>
+                            </xacro:if>
+                            <xacro:unless value="${iface_list}">
+                                <locator>
+                                    <udpv4>
+                                        <address>0.0.0.0</address>
+                                        <port>11811</port>
+                                    </udpv4>
+                                </locator>
+                            </xacro:unless>
                         </metatrafficUnicastLocatorList>
                     </builtin>
